File: PCB/PCB_exo_H_bridge/STM32G4A1REI6_ref_design.kicad_sch (KiCad schematic)
At the start: 37 parts, among them J201 USB_C_Receptacle_USB2.0, J202 Conn_ST_STDC14, SW201 SW_Push, SW202 SW_Push, SW203 SW_Push, U201 STM32G4A1REIx, U202 USBLC6-2SC6, Y202 Crystal_GND24

Commit message: exo done
Parts:
- removed C207: 100n, Capacitor_SMD:C_0402_1005Metric, symbol Device:C_Small
- removed C208, C210: 1u, Capacitor_SMD:C_0603_1608Metric, symbol Device:C_Small
- added C212: 1u, Capacitor_SMD:C_0603_1608Metric, symbol Device:C_Small
- C201: footprint Capacitor_SMD:C_01005_0402Metric -> Capacitor_SMD:C_0402_1005Metric
- C203: renamed from C211; footprint (none) -> Capacitor_SMD:C_0402_1005Metric
- C204: renamed from C212; footprint (none) -> Capacitor_SMD:C_0402_1005Metric
- C208: renamed from C206; MPN (none) -> 885012105020; Vmax (none) -> 6.3V
- C213, C214, C215: footprint (none) -> Capacitor_SMD:C_0402_1005Metric
- D201: renamed from D202; footprint (none) -> LED_SMD:LED_0603_1608Metric
- D202: renamed from D203; footprint (none) -> LED_SMD:LED_0603_1608Metric
- D203: renamed from D201; footprint (none) -> LED_SMD:LED_0603_1608Metric
- J202: footprint (none) -> Connector_PinHeader_1.27mm:PinHeader_2x07_P1.27mm_Vertical_SMD
- L201: footprint (none) -> Inductor_SMD:L_0805_2012Metric
- R201: footprint (none) -> Resistor_SMD:R_0402_1005Metric
- R202: renamed from R208; footprint (none) -> Resistor_SMD:R_0402_1005Metric
- R203: renamed from R209; footprint (none) -> Resistor_SMD:R_0402_1005Metric
- R204: renamed from R207; footprint (none) -> Resistor_SMD:R_0402_1005Metric
- R205: renamed from R210; footprint (none) -> Resistor_SMD:R_0402_1005Metric
- R208: renamed from R205; footprint (none) -> Resistor_SMD:R_0402_1005Metric
- R209: renamed from R206; footprint (none) -> Resistor_SMD:R_0402_1005Metric
- R210: renamed from R204; footprint (none) -> Resistor_SMD:R_0402_1005Metric
- SW201: renamed from SW203; footprint (none) -> Button_Switch_SMD:SW_Push_1P1T_NO_CK_KSC6xxJ
- SW202: footprint (none) -> Button_Switch_SMD:SW_Push_1P1T_NO_CK_KSC6xxJ
- SW203: renamed from SW201; footprint (none) -> Button_Switch_SMD:SW_Push_1P1T_NO_CK_KSC6xxJ
- Y201: renamed from Y202; footprint (none) -> Crystal:Crystal_SMD_3225-4Pin_3.2x2.5mm
- renumbered C203 to C205, C204 to C206, C205 to C207, C209 to C211, R202 to R206, R203 to R207
Connections:
- net +3.3V: no longer U201.G5 (VREF+), U201.H5 (VDDA)
- net +3.3VA: now also U201.G5 (VREF+), U201.H5 (VDDA), C212.1
- net GND: now also R206.2, R207.2, C212.2
- net USR_BTN_1: now also U201.H6 (PB10); no longer U201.A6 (PC12)
- net USR_BTN_2: now also U201.H4 (PB2); no longer U201.A7 (PA15)
- net USR_LED_1: now also U201.A7 (PA15); no longer U201.E8 (PC6)
- net USR_LED_2: now also U201.A6 (PC12); no longer U201.F8 (PB14)
- net USR_LED_3: now also U201.A2 (PB9); no longer U201.G8 (PB12)
- net PWM_CH1N: no longer names the net of U201.B1 (PC13)
- net PWM_CH2N: no longer names the net of U201.E5 (PB0)
Other:
- note removed: "For VREF+"
